File: HW/Roboty_rev2_/MCU.kicad_sch (KiCad schematic)
At the start: 27 parts, among them SW2 BOOT, U1 STM32F446RETx, U4 W25Q32JVSS, Y1 7D026000B01

Commit message: add sd card file library+ new HW version
Parts:
- removed C2: 100n, Capacitor_SMD:C_0603_1608Metric, symbol Device:C
- removed C2: 1u, Capacitor_SMD:C_0603_1608Metric, symbol Device:C
- removed R8: 22R, Resistor_SMD:R_0603_1608Metric, symbol Device:R
- removed U4: W25Q32JVSS, Package_SO:SOIC-8_5.23x5.23mm_P1.27mm, symbol Memory_Flash:W25Q32JVSS
- added C2: 10u, Capacitor_SMD:C_0603_1608Metric, symbol Device:C
- added SW2: BOOT, Button_Switch_SMD:SW_SPST_B3U-1000P, symbol Switch:SW_Push
- C4: value 6.8p -> 12p
- Y1: value 7D026000B01 -> XL7EL89CLI-111YLC-16M
Connections:
- net QSPI_BK1_IO1 is gone; now on net SDIO_D2: U1.51 (PC10)
- net GND: now also C4.1, C2.2, SW2.1; no longer C4.2
- net RST: now also C4.2, SW2.2; no longer C4.1
- net SDIO_D2: no longer U1.27 (PB1)
- net VDDA: now also C2.1
- net at U1.6 (PH1): now also C4.1, Y1.3
- net QSPI_BK1_CLK: no longer names the net of U1.28 (PB2)
- net QSPI_BK1_IO0: no longer names the net of U1.40 (PC9)
- net QSPI_BK1_NCS: no longer names the net of U1.58 (PB6)
- no-connect marks 8 -> 10
Other:
- note removed: "Changez crystal pour un 16MHz adapté en drive au st XC21M4-16.000-F10NLDTL"
- moved on the sheet: C4
